Commit message: Updated mppi track,  made ads_dv  dummy root to have no inertial properties

File: simulation/models/vehicle/ads_dv.xacro (robot description, xacro)
@@ -4,5 +4,5 @@
         <!-- Dummy root link to satisfy KDL (root link must not have inertia) -->
         <link name='base_footprint'>
-            <inertial>
+        <!-- <inertial>
                 <mass>0.0</mass>
                 <inertia>
@@ -14,10 +14,10 @@
                     <izz>0.0</izz>
                 </inertia>
-            </inertial>
+            </inertial> -->
         </link>
         <joint name='base_footprint_to_base_link' type='fixed'>
             <parent>base_footprint</parent>
             <child>base_link</child>
-            <origin xyz="0 0 0" rpy="0 0 0"/>
+            <pose>0 0 0 0 0 0</pose>
         </joint>
         <!-- Base Link -->
